File: Hardware/Kicad/Plaqueta.kicad_pcb (KiCad board)
At the start: 2 copper layers, 41 parts, among them P1 CONN_Entrada, P2 CONN_01X02, SW1 SW_PUSH, SW2 SW_PUSH, SW3 SW_PUSH, SW4 SW_PUSH, SW5 SW_PUSH, U1 MAX680, U2 CD4069, U3 ADG452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

Commit message: Cambios 13/12/16
Other:
- board outline added: 83.6 x 82.2 mm
Changed lines of the file:
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@@
     (links 92)
     (no_connects 0)
-    (area 157.125999 52.733 253.820791 141.892001)
+    (area 157.483476 52.733 241.450001 135.250001)
     (thickness 1.6)
-    (drawings 7)
+    (drawings 5)
     (tracks 297)
     (zones 0)
@@
   )
   (setup
-    (last_trace_width 0.3)
+    (last_trace_width 0.5)
     (user_trace_width 0.3)
     (user_trace_width 0.5)
@@
     (pad 1 np_thru_hole circle (at 0 0) (size 3.5 3.5) (drill 3.5) (layers *.Cu *.Mask F.SilkS))
   )
-  (gr_line (start 157.988 53.34) (end 157.988 135.128) (angle 90) (layer Dwgs.User) (width 0.2))
-  (gr_line (start 241.3 53.34) (end 157.988 53.34) (angle 90) (layer Dwgs.User) (width 0.2))
-  (gr_line (start 241.3 135.128) (end 241.3 53.34) (angle 90) (layer Dwgs.User) (width 0.2))
-  (gr_line (start 157.988 135.128) (end 241.3 135.128) (angle 90) (layer Dwgs.User) (width 0.2))
-  (dimension 82.245451 (width 0.3) (layer Dwgs.User)
-    (gr_text "82,245 mm" (at 247.170791 94.14342 270.1415582) (layer Dwgs.User)
-      (effects (font (size 1.5 1.5) (thickness 0.3)))
-    )
-    (feature1 (pts (xy 241.2492 53.0352) (xy 248.419187 53.017485)))
-    (feature2 (pts (xy 241.4524 135.2804) (xy 248.622387 135.262685)))
-    (crossbar (pts (xy 245.922395 135.269356) (xy 245.719195 53.024156)))
-    (arrow1a (pts (xy 245.719195 53.024156) (xy 246.308397 54.149207)))
-    (arrow1b (pts (xy 245.719195 53.024156) (xy 245.135559 54.152105)))
-    (arrow2a (pts (xy 245.922395 135.269356) (xy 246.506031 134.141407)))
-    (arrow2b (pts (xy 245.922395 135.269356) (xy 245.333193 134.144305)))
-  )
-  (dimension 84.328 (width 0.3) (layer Dwgs.User)
-    (gr_text "84,328 mm" (at 199.39 140.542) (layer Dwgs.User)
-      (effects (font (size 1.5 1.5) (thickness 0.3)))
-    )
-    (feature1 (pts (xy 241.554 135.382) (xy 241.554 141.892)))
-    (feature2 (pts (xy 157.226 135.382) (xy 157.226 141.892)))
-    (crossbar (pts (xy 157.226 139.192) (xy 241.554 139.192)))
-    (arrow1a (pts (xy 241.554 139.192) (xy 240.427496 139.778421)))
-    (arrow1b (pts (xy 241.554 139.192) (xy 240.427496 138.605579)))
-    (arrow2a (pts (xy 157.226 139.192) (xy 158.352504 139.778421)))
-    (arrow2b (pts (xy 157.226 139.192) (xy 158.352504 138.605579)))
-  )
-  (gr_line (start 157.226 135.382) (end 241.3 135.382) (angle 90) (layer Dwgs.User) (width 0.2))
+  (gr_line (start 157.8 135.2) (end 158 135.2) (angle 90) (layer Edge.Cuts) (width 0.1))
+  (gr_line (start 157.8 53) (end 157.8 135.2) (angle 90) (layer Edge.Cuts) (width 0.1))
+  (gr_line (start 241.4 53) (end 157.8 53) (angle 90) (layer Edge.Cuts) (width 0.1))
+  (gr_line (start 241.4 135.2) (end 241.4 53) (angle 90) (layer Edge.Cuts) (width 0.1))
+  (gr_line (start 158 135.2) (end 241.4 135.2) (angle 90) (layer Edge.Cuts) (width 0.1))
   (segment (start 174.498 71.12) (end 174.498 75.9968) (width 0.7) (layer B.Cu) (net 1))
   (segment (start 177.038 71.12) (end 177.038 75.9568) (width 0.7) (layer B.Cu) (net 2))
