File: Hardware/Kicad/Plaqueta.sch (KiCad schematic (older format))
At the start: 37 parts, among them P1 CONN_Entrada, P2 CONN_01X02, SW1 SW_PUSH, SW2 SW_PUSH, SW3 SW_PUSH, SW4 SW_PUSH, SW5 SW_PUSH, U1 MAX680, U2 CD4069, U3 ADG452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

Commit message: Cambios 13/12/16
Changed lines of the file:
@@
 Wire Wire Line
 	1100 5550 1100 5750
+Text Label 8750 2675 0    60   ~ 0
+R12=
+Text Label 8675 2775 0    60   ~ 0
+4k7//1K
+Text Label 5100 4725 0    60   ~ 0
+R9=2K2//8K2
 $EndSCHEMATC
