File: Hardware/Conexiones/conexiones.sch (KiCad schematic (older format))
At the start: 15 parts, among them P1 CONN_20x2, P2 CONN_20x2, P3 CONECTOR_PLAQUETA

Commit message: Corregido
Parts:
- renumbered 5K6 to 1K, 1K to 5K6
Connections:
- net GND: now also 1K.1
- net at P2.1, TH3.2: no longer 1K.1
Changed lines of the file:
@@
 GPIO_GND
 $Comp
-L R 1K
+L R 5K6
 U 1 1 586BF52C
 P 3250 2025
-F 0 "1K" V 3330 2025 50  0000 C CNN
+F 0 "5K6" V 3330 2025 50  0000 C CNN
 F 1 "R" V 3250 2025 50  0000 C CNN
 F 2 "" V 3180 2025 50  0000 C CNN
@@
 $EndComp
 $Comp
-L R 5K6
+L R 1K
 U 1 1 586BF55B
 P 3250 1575
-F 0 "5K6" V 3330 1575 50  0000 C CNN
+F 0 "1K" V 3330 1575 50  0000 C CNN
 F 1 "R" V 3250 1575 50  0000 C CNN
 F 2 "" V 3180 1575 50  0000 C CNN
@@
 	3250 1725 3250 1875
 Wire Wire Line
-	3250 2175 3250 2275
-Wire Wire Line
-	3250 2275 3400 2275
-Wire Wire Line
-	3400 2275 3400 2475
-Connection ~ 3400 2475
-Wire Wire Line
 	4700 1400 4675 1400
 Wire Wire Line
@@
 Wire Wire Line
 	3675 1725 3675 1800
-Wire Wire Line
-	3250 1425 3250 1375
-Wire Wire Line
-	3250 1375 2600 1375
-Wire Wire Line
-	2600 1375 2600 2475
-Connection ~ 2600 2475
 $Comp
 L CONN_01X10 P3
@@
 Connection ~ 1975 4225
 Connection ~ 8350 1925
+Wire Wire Line
+	3250 1425 3250 1375
+Wire Wire Line
+	3250 1375 2600 1375
+Wire Wire Line
+	2600 1375 2600 2575
+Connection ~ 2600 2575
+Wire Wire Line
+	3250 2175 3250 2275
+Wire Wire Line
+	3250 2275 3375 2275
+Wire Wire Line
+	3375 2275 3375 2475
+Connection ~ 3375 2475
 $EndSCHEMATC

Commit message: Corregido
Parts:
- removed TH1, TH2, TH3, TH4: THERMISTOR, symbol THERMISTOR
Connections:
- net +3.3V is gone; now on net VCC: P1.1, P3.2 (P2)
- net +5V is gone; now on net VCC: P1.2, P3.1 (P1)
- net VCC: now also 5K6.2, Display.2 (VDD), P2.1, P2.2, R?.2
Changed lines of the file:
@@
 $EndDescr
-$Comp
-L THERMISTOR TH1
-U 1 1 5868204D
-P 7475 2850
-F 0 "TH1" V 7575 2900 50  0000 C CNN
-F 1 "THERMISTOR" V 7375 2850 50  0000 C BNN
-F 2 "" H 7475 2850 50  0000 C CNN
-F 3 "" H 7475 2850 50  0000 C CNN
-	1    7475 2850
-	1    0    0    -1
-$EndComp
-$Comp
-L THERMISTOR TH2
-U 1 1 586820A1
-P 8900 2875
-F 0 "TH2" V 9000 2925 50  0000 C CNN
-F 1 "THERMISTOR" V 8800 2875 50  0000 C BNN
-F 2 "" H 8900 2875 50  0000 C CNN
-F 3 "" H 8900 2875 50  0000 C CNN
-	1    8900 2875
-	1    0    0    -1
-$EndComp
 $Comp
 L CONN_educiaa P2
@@
 L VCC +3,3V
 U 1 1 58683737
-P 7475 2575
-F 0 "+3,3V" H 7475 2725 50  0000 C CNN
-F 1 "VCC" H 7475 2725 50  0001 C CNN
-F 2 "" H 7475 2575 50  0000 C CNN
-F 3 "" H 7475 2575 50  0000 C CNN
-	1    7475 2575
+P 7475 3125
+F 0 "+3,3V" H 7475 3275 50  0000 C CNN
+F 1 "VCC" H 7475 3275 50  0001 C CNN
+F 2 "" H 7475 3125 50  0000 C CNN
+F 3 "" H 7475 3125 50  0000 C CNN
+	1    7475 3125
 	1    0    0    -1
 $EndComp
@@
 L VCC +5V
 U 1 1 586837D4
-P 8900 2575
-F 0 "+5V" H 8900 2725 50  0000 C CNN
-F 1 "VCC" H 8900 2725 50  0001 C CNN
-F 2 "" H 8900 2575 50  0000 C CNN
-F 3 "" H 8900 2575 50  0000 C CNN
-	1    8900 2575
+P 8900 3125
+F 0 "+5V" H 8900 3275 50  0000 C CNN
+F 1 "VCC" H 8900 3275 50  0001 C CNN
+F 2 "" H 8900 3125 50  0000 C CNN
+F 3 "" H 8900 3125 50  0000 C CNN
+	1    8900 3125
 	1    0    0    -1
 $EndComp
@@
 GPIO_GND
 $Comp
-L THERMISTOR TH3
-U 1 1 586B0052
-P 2350 2025
-F 0 "TH3" V 2450 2075 50  0000 C CNN
-F 1 "THERMISTOR" V 2250 2025 50  0000 C BNN
-F 2 "" H 2350 2025 50  0000 C CNN
-F 3 "" H 2350 2025 50  0000 C CNN
-	1    2350 2025
-	1    0    0    -1
-$EndComp
-$Comp
-L THERMISTOR TH4
-U 1 1 586B0058
-P 3675 2050
-F 0 "TH4" V 3775 2100 50  0000 C CNN
-F 1 "THERMISTOR" V 3575 2050 50  0000 C BNN
-F 2 "" H 3675 2050 50  0000 C CNN
-F 3 "" H 3675 2050 50  0000 C CNN
-	1    3675 2050
-	1    0    0    -1
-$EndComp
-$Comp
 L VCC +3,3V
 U 1 1 586B005E
-P 2350 1700
-F 0 "+3,3V" H 2350 1850 50  0000 C CNN
-F 1 "VCC" H 2350 1850 50  0001 C CNN
-F 2 "" H 2350 1700 50  0000 C CNN
-F 3 "" H 2350 1700 50  0000 C CNN
-	1    2350 1700
+P 2350 2275
+F 0 "+3,3V" H 2350 2425 50  0000 C CNN
+F 1 "VCC" H 2350 2425 50  0001 C CNN
+F 2 "" H 2350 2275 50  0000 C CNN
+F 3 "" H 2350 2275 50  0000 C CNN
+	1    2350 2275
 	1    0    0    -1
 $EndComp
@@
 L VCC +5V
 U 1 1 586B0064
-P 3675 1725
-F 0 "+5V" H 3675 1875 50  0000 C CNN
-F 1 "VCC" H 3675 1875 50  0001 C CNN
-F 2 "" H 3675 1725 50  0000 C CNN
-F 3 "" H 3675 1725 50  0000 C CNN
-	1    3675 1725
+P 3675 2325
+F 0 "+5V" H 3675 2475 50  0000 C CNN
+F 1 "VCC" H 3675 2475 50  0001 C CNN
+F 2 "" H 3675 2325 50  0000 C CNN
+F 3 "" H 3675 2325 50  0000 C CNN
+	1    3675 2325
 	1    0    0    -1
 $EndComp
@@
 	3325 4275 3825 4275
 Wire Wire Line
-	3850 4325 4700 4325
+	3850 4325 4450 4325
+Wire Wire Line
+	4450 4325 4700 4325
 Wire Wire Line
 	3850 4175 3850 4325
@@
 	3325 4175 3850 4175
 Wire Wire Line
-	3875 4200 4700 4200
+	3875 4200 4600 4200
+Wire Wire Line
+	4600 4200 4700 4200
 Wire Wire Line
 	3875 4075 3875 4200
@@
 	3325 4075 3875 4075
 Wire Wire Line
-	3900 4075 4700 4075
+	3900 4075 4525 4075
+Wire Wire Line
+	4525 4075 4700 4075
 Wire Wire Line
 	3900 3975 3900 4075
@@
 	3325 3975 3900 3975
 Wire Wire Line
-	3925 3950 4700 3950
+	3925 3950 4275 3950
+Wire Wire Line
+	4275 3950 4700 3950
 Wire Wire Line
 	3925 3875 3925 3950
@@
 	3325 3875 3925 3875
 Wire Wire Line
-	3950 3825 4700 3825
+	3950 3825 4350 3825
+Wire Wire Line
+	4350 3825 4700 3825
 Wire Wire Line
 	3950 3775 3950 3825
@@
 	3325 3775 3950 3775
 Wire Wire Line
-	3975 3700 4700 3700
+	3975 3700 4225 3700
+Wire Wire Line
+	4225 3700 4700 3700
 Wire Wire Line
 	3975 3675 3975 3700
@@
 	3325 3675 3975 3675
 Wire Wire Line
-	3325 3575 4700 3575
-Wire Wire Line
-	3975 3450 4700 3450
+	3325 3575 4150 3575
+Wire Wire Line
+	4150 3575 4700 3575
+Wire Wire Line
+	3975 3450 4400 3450
+Wire Wire Line
+	4400 3450 4700 3450
 Wire Wire Line
 	3975 3475 3975 3450
@@
 	4700 2325 3725 2325
 Wire Wire Line
-	2200 4375 2625 4375
+	2200 4375 2400 4375
+Wire Wire Line
+	2400 4375 2625 4375
 Wire Wire Line
 	2200 4650 2200 4375
@@
 	2125 4225 2125 4075
 Wire Wire Line
-	1300 4225 2125 4225
+	1300 4225 1975 4225
+Wire Wire Line
+	1975 4225 2125 4225
 Wire Wire Line
 	2100 3975 2625 3975
@@
 	2100 4100 2100 3975
 Wire Wire Line
-	1300 4100 2100 4100
+	1300 4100 1825 4100
+Wire Wire Line
+	1825 4100 2100 4100
 Wire Wire Line
 	2075 3875 2625 3875
@@
 	2075 3975 2075 3875
 Wire Wire Line
-	1300 3975 2075 3975
+	1300 3975 1650 3975
+Wire Wire Line
+	1650 3975 2075 3975
 Wire Wire Line
 	2050 3775 2625 3775
@@
 	875  3725 2025 3725
 Wire Wire Line
-	1275 3575 2625 3575
+	1275 3575 2450 3575
+Wire Wire Line
+	2450 3575 2625 3575
 Wire Wire Line
 	2025 3475 2625 3475
@@
 	850  2425 2225 2425
 Wire Wire Line
-	2250 2575 2625 2575
+	2250 2575 2525 2575
+Wire Wire Line
+	2525 2575 2600 2575
+Wire Wire Line
+	2600 2575 2625 2575
 Wire Wire Line
 	2250 2275 2250 2575
@@
 	850  2275 2250 2275
 Wire Wire Line
-	3675 2475 3675 2300
-Wire Wire Line
-	3325 2475 3675 2475
+	3675 2475 3675 2325
+Wire Wire Line
+	3325 2475 3375 2475
+Wire Wire Line
+	3375 2475 3475 2475
+Wire Wire Line
+	3475 2475 3550 2475
+Wire Wire Line
+	3550 2475 3675 2475
 Wire Wire Line
 	2350 2475 2625 2475
@@
 	2350 2275 2350 2475
 Wire Wire Line
-	2350 1700 2350 1775
-Wire Wire Line
 	8825 5250 8550 5250
 Wire Wire Line
@@
 	9075 4300 9075 4250
 Wire Wire Line
-	9075 4300 10175 4300
+	9075 4300 9425 4300
+Wire Wire Line
+	9425 4300 10175 4300
 Wire Wire Line
 	9050 4150 8550 4150
@@
 	6775 4150 7850 4150
 Wire Wire Line
-	7300 4050 7850 4050
+	7300 4050 7650 4050
+Wire Wire Line
+	7650 4050 7850 4050
 Wire Wire Line
 	7300 4000 7300 4050
@@
 	6225 3525 7400 3525
 Wire Wire Line
-	7475 3100 7475 3350
-Wire Wire Line
-	7475 3350 7850 3350
-Wire Wire Line
-	8550 3350 8900 3350
-Wire Wire Line
-	8900 3350 8900 3125
-Wire Wire Line
-	7475 2575 7475 2600
-Wire Wire Line
-	8900 2575 8900 2625
+	7475 3125 7475 3350
+Wire Wire Line
+	7475 3350 7775 3350
+Wire Wire Line
+	7775 3350 7850 3350
+Wire Wire Line
+	8900 3350 8625 3350
+Wire Wire Line
+	8625 3350 8550 3350
+Wire Wire Line
+	8900 3125 8900 3350
 Wire Wire Line
 	6775 3250 7450 3250
@@
 	4700 1325 4750 1325
 Wire Wire Line
-	4750 1325 4750 1725
+	4750 1325 4750 1475
+Wire Wire Line
+	4750 1475 4750 1725
 Wire Wire Line
 	4750 1475 4700 1475
 Wire Wire Line
-	3250 1725 3250 1875
+	3250 1725 3250 1800
+Wire Wire Line
+	3250 1800 3250 1875
 Wire Wire Line
 	4700 1400 4675 1400
@@
 	3550 1475 3550 2475
 Connection ~ 3550 2475
-Wire Wire Line
-	3675 1725 3675 1800
 $Comp
 L CONN_01X10 P3
@@
 +5V
 Wire Wire Line
-	8025 1025 8550 1025
-Wire Wire Line
-	7950 1125 8550 1125
-Wire Wire Line
-	8025 1225 8550 1225
-Wire Wire Line
-	8150 1325 8550 1325
-Wire Wire Line
-	8150 1425 8550 1425
-Wire Wire Line
-	8150 1525 8550 1525
-Wire Wire Line
-	8150 1625 8550 1625
-Wire Wire Line
-	8150 1725 8550 1725
-Wire Wire Line
-	8150 1825 8550 1825
-Wire Wire Line
-	8150 1925 8550 1925
+	8025 1025 8450 1025
+Wire Wire Line
+	8450 1025 8550 1025
+Wire Wire Line
+	7950 1125 8500 1125
+Wire Wire Line
+	8500 1125 8550 1125
+Wire Wire Line
+	8025 1225 8375 1225
+Wire Wire Line
+	8375 1225 8550 1225
+Wire Wire Line
+	8150 1325 8500 1325
+Wire Wire Line
+	8500 1325 8550 1325
+Wire Wire Line
+	8150 1425 8400 1425
+Wire Wire Line
+	8400 1425 8550 1425
+Wire Wire Line
+	8150 1525 8350 1525
+Wire Wire Line
+	8350 1525 8550 1525
+Wire Wire Line
+	8150 1625 8400 1625
+Wire Wire Line
+	8400 1625 8550 1625
+Wire Wire Line
+	8150 1725 8450 1725
+Wire Wire Line
+	8450 1725 8550 1725
+Wire Wire Line
+	8150 1825 8400 1825
+Wire Wire Line
+	8400 1825 8550 1825
+Wire Wire Line
+	8150 1925 8350 1925
+Wire Wire Line
+	8350 1925 8550 1925
 Wire Wire Line
 	8450 1025 8450 775
